File: STM32_Learning_Shield.kicad_pcb (KiCad board)
At the start: 2 copper layers, 53.3 x 57.6 mm, 44 parts, among them J1 Power, J2 Digital/PWM, J3 Analog, J4 Digital/PWM, J5 XY308-2.54-2P, J6 XY308-2.54-2P, J7 Conn_01x03, J8 Conn_01x03, Q1 2N7002, Q2 2N7002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

Commit message: Add Fiducials
Parts:
- added FID1: Fiducial, Fiducial:Fiducial_1mm_Mask3mm, F.Cu at (117.0, 97.5)
- added FID2: Fiducial, Fiducial:Fiducial_1mm_Mask3mm, F.Cu at (115.0, 50.0)
- added FID3: Fiducial, Fiducial:Fiducial_1mm_Mask3mm, F.Cu at (155.5, 47.5)
- added FID4: Fiducial, Fiducial:Fiducial_1mm_Mask3mm, F.Cu at (140.5, 92.5)
